Commit message: manipulador com a base e o braço faltando a garra

File: braco_description/urdf/braco.xacro (robot description, xacro)
@@ -6,7 +6,7 @@
 <link name="base_link">
   <inertial>
-    <origin rpy="0 0 0" xyz="0.04499629681169275 0.06505950874339432 0.014978663545961009"/>
-    <mass value="0.37092414765363463"/>
-    <inertia ixx="0.00055" ixy="-0.0" ixz="0.0" iyy="0.000279" iyz="-0.0" izz="0.000773"/>
+    <origin rpy="0 0 0" xyz="4.115974110073098e-17 -6.85995685012183e-18 0.018873521383075593"/>
+    <mass value="0.08783440670094944"/>
+    <inertia ixx="0.000167" ixy="-0.0" ixz="0.0" iyy="0.000167" iyz="0.0" izz="0.000245"/>
   </inertial>
   <visual>
@@ -24,12 +24,312 @@
   </collision>
 </link>
+<link name="servo_left_1">
+  <inertial>
+    <origin rpy="0 0 0" xyz="-0.001447315038501595 0.13866693346425074 -0.006915072172979028"/>
+    <mass value="0.25257832542625036"/>
+    <inertia ixx="6.8e-05" ixy="-0.0" ixz="0.0" iyy="4.4e-05" iyz="1e-06" izz="4.1e-05"/>
+  </inertial>
+  <visual>
+    <origin rpy="0 0 0" xyz="-0.002899 0.089641 -0.108609"/>
+    <geometry>
+      <mesh filename="package://braco_description/meshes/servo_left_1.stl" scale="0.001 0.001 0.001"/>
+    </geometry>
+    <material name="silver"/>
+  </visual>
+  <collision>
+    <origin rpy="0 0 0" xyz="-0.002899 0.089641 -0.108609"/>
+    <geometry>
+      <mesh filename="package://braco_description/meshes/servo_left_1.stl" scale="0.001 0.001 0.001"/>
+    </geometry>
+  </collision>
+</link>
+<link name="servo_right_1">
+  <inertial>
+    <origin rpy="0 0 0" xyz="0.06544272704404513 -0.13866641850044178 0.07250492782702278"/>
+    <mass value="0.25257832542625036"/>
+    <inertia ixx="6.8e-05" ixy="-0.0" ixz="-0.0" iyy="4.4e-05" iyz="-1e-06" izz="4.1e-05"/>
+  </inertial>
+  <visual>
+    <origin rpy="0 0 0" xyz="0.064 -0.090439 -0.029189"/>
+    <geometry>
+      <mesh filename="package://braco_description/meshes/servo_right_1.stl" scale="0.001 0.001 0.001"/>
+    </geometry>
+    <material name="silver"/>
+  </visual>
+  <collision>
+    <origin rpy="0 0 0" xyz="0.064 -0.090439 -0.029189"/>
+    <geometry>
+      <mesh filename="package://braco_description/meshes/servo_right_1.stl" scale="0.001 0.001 0.001"/>
+    </geometry>
+  </collision>
+</link>
+<link name="Center_arm_v1_1">
+  <inertial>
+    <origin rpy="0 0 0" xyz="-0.000706868206479333 0.009887184158138773 -0.057802053392263214"/>
+    <mass value="0.24743903954578314"/>
+    <inertia ixx="0.000566" ixy="0.0" ixz="-5e-06" iyy="0.000605" iyz="-0.0" izz="7.6e-05"/>
+  </inertial>
+  <visual>
+    <origin rpy="0 0 0" xyz="-0.168543 0.011691 -0.190905"/>
+    <geometry>
+      <mesh filename="package://braco_description/meshes/Center_arm_v1_1.stl" scale="0.001 0.001 0.001"/>
+    </geometry>
+    <material name="silver"/>
+  </visual>
+  <collision>
+    <origin rpy="0 0 0" xyz="-0.168543 0.011691 -0.190905"/>
+    <geometry>
+      <mesh filename="package://braco_description/meshes/Center_arm_v1_1.stl" scale="0.001 0.001 0.001"/>
+    </geometry>
+  </collision>
+</link>
+<link name="Center_arm_bearing_guide_v1_1">
+  <inertial>
+    <origin rpy="0 0 0" xyz="-0.00848571695628475 0.0032219623568815314 0.008485254227916017"/>
+    <mass value="0.0033035453927957375"/>
+    <inertia ixx="0.0" ixy="-0.0" ixz="0.0" iyy="0.0" iyz="-0.0" izz="0.0"/>
+  </inertial>
+  <visual>
+    <origin rpy="0 0 0" xyz="-0.177029 -0.008309 -0.18242"/>
+    <geometry>
+      <mesh filename="package://braco_description/meshes/Center_arm_bearing_guide_v1_1.stl" scale="0.001 0.001 0.001"/>
+    </geometry>
+    <material name="silver"/>
+  </visual>
+  <collision>
+    <origin rpy="0 0 0" xyz="-0.177029 -0.008309 -0.18242"/>
+    <geometry>
+      <mesh filename="package://braco_description/meshes/Center_arm_bearing_guide_v1_1.stl" scale="0.001 0.001 0.001"/>
+    </geometry>
+  </collision>
+</link>
+<link name="Center_arm_bearing_guide_v1__1__1">
+  <inertial>
+    <origin rpy="0 0 0" xyz="-0.00848571695625519 0.0032219623568797325 -0.008485745772046693"/>
+    <mass value="0.0033035453927957375"/>
+    <inertia ixx="0.0" ixy="0.0" ixz="0.0" iyy="0.0" iyz="0.0" izz="0.0"/>
+  </inertial>
+  <visual>
+    <origin rpy="0 0 0" xyz="-0.177029 -0.008309 -0.081891"/>
+    <geometry>
+      <mesh filename="package://braco_description/meshes/Center_arm_bearing_guide_v1__1__1.stl" scale="0.001 0.001 0.001"/>
+    </geometry>
+    <material name="silver"/>
+  </visual>
+  <collision>
+    <origin rpy="0 0 0" xyz="-0.177029 -0.008309 -0.081891"/>
+    <geometry>
+      <mesh filename="package://braco_description/meshes/Center_arm_bearing_guide_v1__1__1.stl" scale="0.001 0.001 0.001"/>
+    </geometry>
+  </collision>
+</link>
+<link name="Center_arm_bearing_guide_clamp_v1_1">
+  <inertial>
+    <origin rpy="0 0 0" xyz="2.8304380533805684e-07 0.0016578450305458174 2.542279526340785e-07"/>
+    <mass value="0.00026744770959091237"/>
+    <inertia ixx="0.0" ixy="-0.0" ixz="-0.0" iyy="0.0" iyz="0.0" izz="0.0"/>
+  </inertial>
+  <visual>
+    <origin rpy="0 0 0" xyz="-0.168543 -0.021709 -0.190905"/>
+    <geometry>
+      <mesh filename="package://braco_description/meshes/Center_arm_bearing_guide_clamp_v1_1.stl" scale="0.001 0.001 0.001"/>
+    </geometry>
+    <material name="silver"/>
+  </visual>
+  <collision>
+    <origin rpy="0 0 0" xyz="-0.168543 -0.021709 -0.190905"/>
+    <geometry>
+      <mesh filename="package://braco_description/meshes/Center_arm_bearing_guide_clamp_v1_1.stl" scale="0.001 0.001 0.001"/>
+    </geometry>
+  </collision>
+</link>
+<link name="ombro_1">
+  <inertial>
+    <origin rpy="0 0 0" xyz="0.08425500605814486 0.024406441382174574 0.03992975695830696"/>
+    <mass value="0.488316525379642"/>
+    <inertia ixx="0.000841" ixy="-3.4e-05" ixz="-0.000637" iyy="0.001965" iyz="-1.6e-05" izz="0.001884"/>
+  </inertial>
+  <visual>
+    <origin rpy="0 0 0" xyz="-0.001443 0.023001 -0.11167"/>
+    <geometry>
+      <mesh filename="package://braco_description/meshes/ombro_1.stl" scale="0.001 0.001 0.001"/>
+    </geometry>
+    <material name="silver"/>
+  </visual>
+  <collision>
+    <origin rpy="0 0 0" xyz="-0.001443 0.023001 -0.11167"/>
+    <geometry>
+      <mesh filename="package://braco_description/meshes/ombro_1.stl" scale="0.001 0.001 0.001"/>
+    </geometry>
+  </collision>
+</link>
+<link name="Bearing_holder_v1_elbow_1">
+  <inertial>
+    <origin rpy="0 0 0" xyz="3.194508534920537e-07 -0.004478970044736082 3.475102374472794e-07"/>
+    <mass value="0.004555197598329582"/>
+    <inertia ixx="0.0" ixy="0.0" ixz="-0.0" iyy="1e-06" iyz="0.0" izz="1e-06"/>
+  </inertial>
+  <visual>
+    <origin rpy="0 0 0" xyz="-0.168619 -0.023799 -0.190897"/>
+    <geometry>
+      <mesh filename="package://braco_description/meshes/Bearing_holder_v1_elbow_1.stl" scale="0.001 0.001 0.001"/>
+    </geometry>
+    <material name="silver"/>
+  </visual>
+  <collision>
+    <origin rpy="0 0 0" xyz="-0.168619 -0.023799 -0.190897"/>
+    <geometry>
+      <mesh filename="package://braco_description/meshes/Bearing_holder_v1_elbow_1.stl" scale="0.001 0.001 0.001"/>
+    </geometry>
+  </collision>
+</link>
+<link name="servo_elbow_1">
+  <inertial>
+    <origin rpy="0 0 0" xyz="0.11594994326799526 0.2079486078632405 -0.05134182605242854"/>
+    <mass value="0.2525786066068201"/>
+    <inertia ixx="4.6e-05" ixy="-0.0" ixz="-1.1e-05" iyy="4.4e-05" iyz="-0.0" izz="6.3e-05"/>
+  </inertial>
+  <visual>
+    <origin rpy="0 0 0" xyz="-0.043552 0.244866 -0.238031"/>
+    <geometry>
+      <mesh filename="package://braco_description/meshes/servo_elbow_1.stl" scale="0.001 0.001 0.001"/>
+    </geometry>
+    <material name="silver"/>
+  </visual>
+  <collision>
+    <origin rpy="0 0 0" xyz="-0.043552 0.244866 -0.238031"/>
+    <geometry>
+      <mesh filename="package://braco_description/meshes/servo_elbow_1.stl" scale="0.001 0.001 0.001"/>
+    </geometry>
+  </collision>
+</link>
+<link name="servo_punho_rot_1">
+  <inertial>
+    <origin rpy="0 0 0" xyz="0.12129196273098862 -0.10986496796742763 -0.2166544630735875"/>
+    <mass value="0.25257832542625036"/>
+    <inertia ixx="4.4e-05" ixy="-0.0" ixz="1e-06" iyy="6.8e-05" iyz="0.0" izz="4.1e-05"/>
+  </inertial>
+  <visual>
+    <origin rpy="0 0 0" xyz="-0.108674 -0.110262 -0.29972"/>
+    <geometry>
+      <mesh filename="package://braco_description/meshes/servo_punho_rot_1.stl" scale="0.001 0.001 0.001"/>
+    </geometry>
+    <material name="silver"/>
+  </visual>
+  <collision>
+    <origin rpy="0 0 0" xyz="-0.108674 -0.110262 -0.29972"/>
+    <geometry>
+      <mesh filename="package://braco_description/meshes/servo_punho_rot_1.stl" scale="0.001 0.001 0.001"/>
+    </geometry>
+  </collision>
+</link>
+<link name="servo_punho_xy_1">
+  <inertial>
+    <origin rpy="0 0 0" xyz="0.00997632381475877 -0.025226418500439357 2.822880096897684e-07"/>
+    <mass value="0.25257832542625036"/>
+    <inertia ixx="4.1e-05" ixy="1e-06" ixz="0.0" iyy="4.4e-05" iyz="-0.0" izz="6.8e-05"/>
+  </inertial>
+  <visual>
+    <origin rpy="0 0 0" xyz="-0.168543 0.011691 -0.073405"/>
+    <geometry>
+      <mesh filename="package://braco_description/meshes/servo_punho_xy_1.stl" scale="0.001 0.001 0.001"/>
+    </geometry>
+    <material name="silver"/>
+  </visual>
+  <collision>
+    <origin rpy="0 0 0" xyz="-0.168543 0.011691 -0.073405"/>
+    <geometry>
+      <mesh filename="package://braco_description/meshes/servo_punho_xy_1.stl" scale="0.001 0.001 0.001"/>
+    </geometry>
+  </collision>
+</link>
+<link name="punho_1">
+  <inertial>
+    <origin rpy="0 0 0" xyz="-0.12859312744504042 0.10167389824420814 0.028959375746381716"/>
+    <mass value="0.21880690583277723"/>
+    <inertia ixx="0.000235" ixy="1.1e-05" ixz="-7e-06" iyy="0.000273" iyz="0.0" izz="0.000371"/>
+  </inertial>
+  <visual>
+    <origin rpy="0 0 0" xyz="-0.333684 0.099028 -0.045405"/>
+    <geometry>
+      <mesh filename="package://braco_description/meshes/punho_1.stl" scale="0.001 0.001 0.001"/>
+    </geometry>
+    <material name="silver"/>
+  </visual>
+  <collision>
+    <origin rpy="0 0 0" xyz="-0.333684 0.099028 -0.045405"/>
+    <geometry>
+      <mesh filename="package://braco_description/meshes/punho_1.stl" scale="0.001 0.001 0.001"/>
+    </geometry>
+  </collision>
+</link>
+<link name="Center_arm_bearing_guide_clamp_v1_punho_1">
+  <inertial>
+    <origin rpy="0 0 0" xyz="2.830437085266091e-07 0.0016578450305452658 2.542280482520365e-07"/>
+    <mass value="0.00026744770959091237"/>
+    <inertia ixx="0.0" ixy="0.0" ixz="0.0" iyy="0.0" iyz="-0.0" izz="0.0"/>
+  </inertial>
+  <visual>
+    <origin rpy="0 0 0" xyz="-0.168543 -0.021709 -0.073405"/>
+    <geometry>
+      <mesh filename="package://braco_description/meshes/Center_arm_bearing_guide_clamp_v1_punho_1.stl" scale="0.001 0.001 0.001"/>
+    </geometry>
+    <material name="silver"/>
+  </visual>
+  <collision>
+    <origin rpy="0 0 0" xyz="-0.168543 -0.021709 -0.073405"/>
+    <geometry>
+      <mesh filename="package://braco_description/meshes/Center_arm_bearing_guide_clamp_v1_punho_1.stl" scale="0.001 0.001 0.001"/>
+    </geometry>
+  </collision>
+</link>
+<link name="Bearing_holder_v1_punho_1">
+  <inertial>
+    <origin rpy="0 0 0" xyz="-3.6128669958501725e-07 -0.003920514991448638 -4.922626540976305e-07"/>
+    <mass value="0.004555197598329582"/>
+    <inertia ixx="0.0" ixy="0.0" ixz="0.0" iyy="1e-06" iyz="0.0" izz="1e-06"/>
+  </inertial>
+  <visual>
+    <origin rpy="0 0 0" xyz="-0.168883 -0.023799 -0.073408"/>
+    <geometry>
+      <mesh filename="package://braco_description/meshes/Bearing_holder_v1_punho_1.stl" scale="0.001 0.001 0.001"/>
+    </geometry>
+    <material name="silver"/>
+  </visual>
+  <collision>
+    <origin rpy="0 0 0" xyz="-0.168883 -0.023799 -0.073408"/>
+    <geometry>
+      <mesh filename="package://braco_description/meshes/Bearing_holder_v1_punho_1.stl" scale="0.001 0.001 0.001"/>
+    </geometry>
+  </collision>
+</link>
+<link name="tampa_1">
+  <inertial>
+    <origin rpy="0 0 0" xyz="-6.348378147066116e-06 -1.751400612895522e-06 0.0014999999999999875"/>
+    <mass value="0.03288605303938267"/>
+    <inertia ixx="2.7e-05" ixy="0.0" ixz="-0.0" iyy="2.7e-05" iyz="0.0" izz="5.4e-05"/>
+  </inertial>
+  <visual>
+    <origin rpy="0 0 0" xyz="-0.0 0.0 -0.0655"/>
+    <geometry>
+      <mesh filename="package://braco_description/meshes/tampa_1.stl" scale="0.001 0.001 0.001"/>
+    </geometry>
+    <material name="silver"/>
+  </visual>
+  <collision>
+    <origin rpy="0 0 0" xyz="-0.0 0.0 -0.0655"/>
+    <geometry>
+      <mesh filename="package://braco_description/meshes/tampa_1.stl" scale="0.001 0.001 0.001"/>
+    </geometry>
+  </collision>
+</link>
 <link name="Base_servo_mount_left_1">
   <inertial>
-    <origin rpy="0 0 0" xyz="-0.015875047506620873 0.00020585580724742647 0.042452933406571636"/>
+    <origin rpy="0 0 0" xyz="-0.015874540487837988 0.00020637077105250395 0.042452933406575036"/>
     <mass value="0.04710420541299449"/>
     <inertia ixx="2.1e-05" ixy="0.0" ixz="0.0" iyy="3.9e-05" iyz="0.0" izz="2e-05"/>
   </inertial>
   <visual>
-    <origin rpy="0 0 0" xyz="-0.06232 -0.101811 -0.03"/>
+    <origin rpy="0 0 0" xyz="-0.017324 -0.037609 -0.0685"/>
     <geometry>
       <mesh filename="package://braco_description/meshes/Base_servo_mount_left_1.stl" scale="0.001 0.001 0.001"/>
@@ -38,5 +338,5 @@
   </visual>
   <collision>
-    <origin rpy="0 0 0" xyz="-0.06232 -0.101811 -0.03"/>
+    <origin rpy="0 0 0" xyz="-0.017324 -0.037609 -0.0685"/>
     <geometry>
       <mesh filename="package://braco_description/meshes/Base_servo_mount_left_1.stl" scale="0.001 0.001 0.001"/>
@@ -44,52 +344,12 @@
   </collision>
 </link>
-<link name="servo_left_1">
-  <inertial>
-    <origin rpy="0 0 0" xyz="-0.04644282205728416 0.10016641850044598 -0.07111707217298194"/>
-    <mass value="0.25257832542625036"/>
-    <inertia ixx="6.8e-05" ixy="-0.0" ixz="0.0" iyy="4.4e-05" iyz="1e-06" izz="4.1e-05"/>
-  </inertial>
-  <visual>
-    <origin rpy="0 0 0" xyz="-0.09289 -0.013061 -0.134311"/>
-    <geometry>
-      <mesh filename="package://braco_description/meshes/servo_left_1.stl" scale="0.001 0.001 0.001"/>
-    </geometry>
-    <material name="silver"/>
-  </visual>
-  <collision>
-    <origin rpy="0 0 0" xyz="-0.09289 -0.013061 -0.134311"/>
-    <geometry>
-      <mesh filename="package://braco_description/meshes/servo_left_1.stl" scale="0.001 0.001 0.001"/>
-    </geometry>
-  </collision>
-</link>
-<link name="servo_right_1">
-  <inertial>
-    <origin rpy="0 0 0" xyz="0.11044723406282062 -0.10016693346424686 0.008302927827013674"/>
-    <mass value="0.25257832542625036"/>
-    <inertia ixx="6.8e-05" ixy="-0.0" ixz="-0.0" iyy="4.4e-05" iyz="-1e-06" izz="4.1e-05"/>
-  </inertial>
-  <visual>
-    <origin rpy="0 0 0" xyz="0.064 -0.116141 -0.054891"/>
-    <geometry>
-      <mesh filename="package://braco_description/meshes/servo_right_1.stl" scale="0.001 0.001 0.001"/>
-    </geometry>
-    <material name="silver"/>
-  </visual>
-  <collision>
-    <origin rpy="0 0 0" xyz="0.064 -0.116141 -0.054891"/>
-    <geometry>
-      <mesh filename="package://braco_description/meshes/servo_right_1.stl" scale="0.001 0.001 0.001"/>
-    </geometry>
-  </collision>
-</link>
 <link name="Base_servo_mount_right_v1_1">
   <inertial>
-    <origin rpy="0 0 0" xyz="-0.01587454048784174 -0.00020637077104875348 0.04245293340656735"/>
+    <origin rpy="0 0 0" xyz="-0.015875047506617494 -0.00020585580724314517 0.04245293340657591"/>
     <mass value="0.04710420541299451"/>
-    <inertia ixx="2.1e-05" ixy="0.0" ixz="-0.0" iyy="3.9e-05" iyz="-0.0" izz="2e-05"/>
-  </inertial>
-  <visual>
-    <origin rpy="0 0 0" xyz="-0.062324 -0.027391 -0.03"/>
+    <inertia ixx="2.1e-05" ixy="-0.0" ixz="-0.0" iyy="3.9e-05" iyz="-0.0" izz="2e-05"/>
+  </inertial>
+  <visual>
+    <origin rpy="0 0 0" xyz="-0.01732 0.036811 -0.0685"/>
     <geometry>
       <mesh filename="package://braco_description/meshes/Base_servo_mount_right_v1_1.stl" scale="0.001 0.001 0.001"/>
@@ -98,5 +358,5 @@
   </visual>
   <collision>
-    <origin rpy="0 0 0" xyz="-0.062324 -0.027391 -0.03"/>
+    <origin rpy="0 0 0" xyz="-0.01732 0.036811 -0.0685"/>
     <geometry>
       <mesh filename="package://braco_description/meshes/Base_servo_mount_right_v1_1.stl" scale="0.001 0.001 0.001"/>
@@ -104,200 +364,117 @@
   </collision>
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