Commit message: Manipulador sem motor na base

File: braco_description/urdf/braco.xacro (robot description, xacro)
@@ -6,7 +6,7 @@
 <link name="base_link">
   <inertial>
-    <origin rpy="0 0 0" xyz="4.115974110073098e-17 -6.85995685012183e-18 0.018873521383075593"/>
+    <origin rpy="0 0 0" xyz="1.7530925309878173e-17 -4.54861709507948e-18 0.02187352138307566"/>
     <mass value="0.08783440670094944"/>
-    <inertia ixx="0.000167" ixy="-0.0" ixz="0.0" iyy="0.000167" iyz="0.0" izz="0.000245"/>
+    <inertia ixx="0.000167" ixy="0.0" ixz="-0.0" iyy="0.000167" iyz="0.0" izz="0.000245"/>
   </inertial>
   <visual>
@@ -26,10 +26,10 @@
 <link name="servo_left_1">
   <inertial>
-    <origin rpy="0 0 0" xyz="-0.001447315038501595 0.13866693346425074 -0.006915072172979028"/>
+    <origin rpy="0 0 0" xyz="-0.0014473150385015854 0.1421669334642504 -0.006915072172979028"/>
     <mass value="0.25257832542625036"/>
     <inertia ixx="6.8e-05" ixy="-0.0" ixz="0.0" iyy="4.4e-05" iyz="1e-06" izz="4.1e-05"/>
   </inertial>
   <visual>
-    <origin rpy="0 0 0" xyz="-0.002899 0.089641 -0.108609"/>
+    <origin rpy="0 0 0" xyz="-0.002899 0.093141 -0.112109"/>
     <geometry>
       <mesh filename="package://braco_description/meshes/servo_left_1.stl" scale="0.001 0.001 0.001"/>
@@ -38,5 +38,5 @@
   </visual>
   <collision>
-    <origin rpy="0 0 0" xyz="-0.002899 0.089641 -0.108609"/>
+    <origin rpy="0 0 0" xyz="-0.002899 0.093141 -0.112109"/>
     <geometry>
       <mesh filename="package://braco_description/meshes/servo_left_1.stl" scale="0.001 0.001 0.001"/>
@@ -46,10 +46,10 @@
 <link name="servo_right_1">
   <inertial>
-    <origin rpy="0 0 0" xyz="0.06544272704404513 -0.13866641850044178 0.07250492782702278"/>
+    <origin rpy="0 0 0" xyz="0.06544272704404532 -0.14216641850044148 0.07250492782702281"/>
     <mass value="0.25257832542625036"/>
     <inertia ixx="6.8e-05" ixy="-0.0" ixz="-0.0" iyy="4.4e-05" iyz="-1e-06" izz="4.1e-05"/>
   </inertial>
   <visual>
-    <origin rpy="0 0 0" xyz="0.064 -0.090439 -0.029189"/>
+    <origin rpy="0 0 0" xyz="0.064 -0.093939 -0.032689"/>
     <geometry>
       <mesh filename="package://braco_description/meshes/servo_right_1.stl" scale="0.001 0.001 0.001"/>
@@ -58,5 +58,5 @@
   </visual>
   <collision>
-    <origin rpy="0 0 0" xyz="0.064 -0.090439 -0.029189"/>
+    <origin rpy="0 0 0" xyz="0.064 -0.093939 -0.032689"/>
     <geometry>
       <mesh filename="package://braco_description/meshes/servo_right_1.stl" scale="0.001 0.001 0.001"/>
@@ -66,10 +66,10 @@
 <link name="Center_arm_v1_1">
   <inertial>
-    <origin rpy="0 0 0" xyz="-0.000706868206479333 0.009887184158138773 -0.057802053392263214"/>
+    <origin rpy="0 0 0" xyz="-0.0007068682064791942 0.009887184158139134 -0.05780205339226316"/>
     <mass value="0.24743903954578314"/>
     <inertia ixx="0.000566" ixy="0.0" ixz="-5e-06" iyy="0.000605" iyz="-0.0" izz="7.6e-05"/>
   </inertial>
   <visual>
-    <origin rpy="0 0 0" xyz="-0.168543 0.011691 -0.190905"/>
+    <origin rpy="0 0 0" xyz="-0.168543 0.011691 -0.194405"/>
     <geometry>
       <mesh filename="package://braco_description/meshes/Center_arm_v1_1.stl" scale="0.001 0.001 0.001"/>
@@ -78,5 +78,5 @@
   </visual>
   <collision>
-    <origin rpy="0 0 0" xyz="-0.168543 0.011691 -0.190905"/>
+    <origin rpy="0 0 0" xyz="-0.168543 0.011691 -0.194405"/>
     <geometry>
       <mesh filename="package://braco_description/meshes/Center_arm_v1_1.stl" scale="0.001 0.001 0.001"/>
@@ -86,10 +86,10 @@
 <link name="Center_arm_bearing_guide_v1_1">
   <inertial>
-    <origin rpy="0 0 0" xyz="-0.00848571695628475 0.0032219623568815314 0.008485254227916017"/>
+    <origin rpy="0 0 0" xyz="-0.008485716956284667 0.003221962356881842 0.008485254227916045"/>
     <mass value="0.0033035453927957375"/>
     <inertia ixx="0.0" ixy="-0.0" ixz="0.0" iyy="0.0" iyz="-0.0" izz="0.0"/>
   </inertial>
   <visual>
-    <origin rpy="0 0 0" xyz="-0.177029 -0.008309 -0.18242"/>
+    <origin rpy="0 0 0" xyz="-0.177029 -0.008309 -0.18592"/>
     <geometry>
       <mesh filename="package://braco_description/meshes/Center_arm_bearing_guide_v1_1.stl" scale="0.001 0.001 0.001"/>
@@ -98,5 +98,5 @@
   </visual>
   <collision>
-    <origin rpy="0 0 0" xyz="-0.177029 -0.008309 -0.18242"/>
+    <origin rpy="0 0 0" xyz="-0.177029 -0.008309 -0.18592"/>
     <geometry>
       <mesh filename="package://braco_description/meshes/Center_arm_bearing_guide_v1_1.stl" scale="0.001 0.001 0.001"/>
@@ -106,10 +106,10 @@
 <link name="Center_arm_bearing_guide_v1__1__1">
   <inertial>
-    <origin rpy="0 0 0" xyz="-0.00848571695625519 0.0032219623568797325 -0.008485745772046693"/>
+    <origin rpy="0 0 0" xyz="-0.008485716956255163 0.003221962356880064 -0.008485745772046652"/>
     <mass value="0.0033035453927957375"/>
-    <inertia ixx="0.0" ixy="0.0" ixz="0.0" iyy="0.0" iyz="0.0" izz="0.0"/>
-  </inertial>
-  <visual>
-    <origin rpy="0 0 0" xyz="-0.177029 -0.008309 -0.081891"/>
+    <inertia ixx="0.0" ixy="0.0" ixz="-0.0" iyy="0.0" iyz="0.0" izz="0.0"/>
+  </inertial>
+  <visual>
+    <origin rpy="0 0 0" xyz="-0.177029 -0.008309 -0.085391"/>
     <geometry>
       <mesh filename="package://braco_description/meshes/Center_arm_bearing_guide_v1__1__1.stl" scale="0.001 0.001 0.001"/>
@@ -118,5 +118,5 @@
   </visual>
   <collision>
-    <origin rpy="0 0 0" xyz="-0.177029 -0.008309 -0.081891"/>
+    <origin rpy="0 0 0" xyz="-0.177029 -0.008309 -0.085391"/>
     <geometry>
       <mesh filename="package://braco_description/meshes/Center_arm_bearing_guide_v1__1__1.stl" scale="0.001 0.001 0.001"/>
@@ -126,10 +126,10 @@
 <link name="Center_arm_bearing_guide_clamp_v1_1">
   <inertial>
-    <origin rpy="0 0 0" xyz="2.8304380533805684e-07 0.0016578450305458174 2.542279526340785e-07"/>
+    <origin rpy="0 0 0" xyz="2.8304380533805684e-07 0.0016578450305459944 2.542279528283675e-07"/>
     <mass value="0.00026744770959091237"/>
-    <inertia ixx="0.0" ixy="-0.0" ixz="-0.0" iyy="0.0" iyz="0.0" izz="0.0"/>
-  </inertial>
-  <visual>
-    <origin rpy="0 0 0" xyz="-0.168543 -0.021709 -0.190905"/>
+    <inertia ixx="0.0" ixy="-0.0" ixz="0.0" iyy="0.0" iyz="0.0" izz="0.0"/>
+  </inertial>
+  <visual>
+    <origin rpy="0 0 0" xyz="-0.168543 -0.021709 -0.194405"/>
     <geometry>
       <mesh filename="package://braco_description/meshes/Center_arm_bearing_guide_clamp_v1_1.stl" scale="0.001 0.001 0.001"/>
@@ -138,5 +138,5 @@
   </visual>
   <collision>
-    <origin rpy="0 0 0" xyz="-0.168543 -0.021709 -0.190905"/>
+    <origin rpy="0 0 0" xyz="-0.168543 -0.021709 -0.194405"/>
     <geometry>
       <mesh filename="package://braco_description/meshes/Center_arm_bearing_guide_clamp_v1_1.stl" scale="0.001 0.001 0.001"/>
@@ -146,10 +146,10 @@
 <link name="ombro_1">
   <inertial>
-    <origin rpy="0 0 0" xyz="0.08425500605814486 0.024406441382174574 0.03992975695830696"/>
+    <origin rpy="0 0 0" xyz="0.08425500605814484 0.024406441382175036 0.039929756958307056"/>
     <mass value="0.488316525379642"/>
     <inertia ixx="0.000841" ixy="-3.4e-05" ixz="-0.000637" iyy="0.001965" iyz="-1.6e-05" izz="0.001884"/>
   </inertial>
   <visual>
-    <origin rpy="0 0 0" xyz="-0.001443 0.023001 -0.11167"/>
+    <origin rpy="0 0 0" xyz="-0.001443 0.023001 -0.11517"/>
     <geometry>
       <mesh filename="package://braco_description/meshes/ombro_1.stl" scale="0.001 0.001 0.001"/>
@@ -158,5 +158,5 @@
   </visual>
   <collision>
-    <origin rpy="0 0 0" xyz="-0.001443 0.023001 -0.11167"/>
+    <origin rpy="0 0 0" xyz="-0.001443 0.023001 -0.11517"/>
     <geometry>
       <mesh filename="package://braco_description/meshes/ombro_1.stl" scale="0.001 0.001 0.001"/>
@@ -166,10 +166,10 @@
 <link name="servo_elbow_1">
   <inertial>
-    <origin rpy="0 0 0" xyz="0.11594994326799526 0.2079486078632405 -0.05134182605242854"/>
+    <origin rpy="0 0 0" xyz="0.11594994326799538 0.20794860786324101 -0.05484182605242849"/>
     <mass value="0.2525786066068201"/>
     <inertia ixx="4.6e-05" ixy="-0.0" ixz="-1.1e-05" iyy="4.4e-05" iyz="-0.0" izz="6.3e-05"/>
   </inertial>
   <visual>
-    <origin rpy="0 0 0" xyz="-0.043552 0.244866 -0.238031"/>
+    <origin rpy="0 0 0" xyz="-0.043552 0.244866 -0.245031"/>
     <geometry>
       <mesh filename="package://braco_description/meshes/servo_elbow_1.stl" scale="0.001 0.001 0.001"/>
@@ -178,5 +178,5 @@
   </visual>
   <collision>
-    <origin rpy="0 0 0" xyz="-0.043552 0.244866 -0.238031"/>
+    <origin rpy="0 0 0" xyz="-0.043552 0.244866 -0.245031"/>
     <geometry>
       <mesh filename="package://braco_description/meshes/servo_elbow_1.stl" scale="0.001 0.001 0.001"/>
@@ -186,10 +186,10 @@
 <link name="servo_punho_rot_1">
   <inertial>
-    <origin rpy="0 0 0" xyz="0.12129196273098862 -0.10986496796742763 -0.2166544630735875"/>
+    <origin rpy="0 0 0" xyz="0.12479196273098876 -0.10986496796742719 -0.2166544630735875"/>
     <mass value="0.25257832542625036"/>
     <inertia ixx="4.4e-05" ixy="-0.0" ixz="1e-06" iyy="6.8e-05" iyz="0.0" izz="4.1e-05"/>
   </inertial>
   <visual>
-    <origin rpy="0 0 0" xyz="-0.108674 -0.110262 -0.29972"/>
+    <origin rpy="0 0 0" xyz="-0.105174 -0.110262 -0.30322"/>
     <geometry>
       <mesh filename="package://braco_description/meshes/servo_punho_rot_1.stl" scale="0.001 0.001 0.001"/>
@@ -198,5 +198,5 @@
   </visual>
   <collision>
-    <origin rpy="0 0 0" xyz="-0.108674 -0.110262 -0.29972"/>
+    <origin rpy="0 0 0" xyz="-0.105174 -0.110262 -0.30322"/>
     <geometry>
       <mesh filename="package://braco_description/meshes/servo_punho_rot_1.stl" scale="0.001 0.001 0.001"/>
@@ -206,10 +206,10 @@
 <link name="servo_punho_xy_1">
   <inertial>
-    <origin rpy="0 0 0" xyz="0.00997632381475877 -0.025226418500439357 2.822880096897684e-07"/>
+    <origin rpy="0 0 0" xyz="0.009976323814758825 -0.025226418500438767 2.8228800974527957e-07"/>
     <mass value="0.25257832542625036"/>
     <inertia ixx="4.1e-05" ixy="1e-06" ixz="0.0" iyy="4.4e-05" iyz="-0.0" izz="6.8e-05"/>
   </inertial>
   <visual>
-    <origin rpy="0 0 0" xyz="-0.168543 0.011691 -0.073405"/>
+    <origin rpy="0 0 0" xyz="-0.168543 0.011691 -0.076905"/>
     <geometry>
       <mesh filename="package://braco_description/meshes/servo_punho_xy_1.stl" scale="0.001 0.001 0.001"/>
@@ -218,5 +218,5 @@
   </visual>
   <collision>
-    <origin rpy="0 0 0" xyz="-0.168543 0.011691 -0.073405"/>
+    <origin rpy="0 0 0" xyz="-0.168543 0.011691 -0.076905"/>
     <geometry>
       <mesh filename="package://braco_description/meshes/servo_punho_xy_1.stl" scale="0.001 0.001 0.001"/>
@@ -226,10 +226,10 @@
 <link name="punho_1">
   <inertial>
-    <origin rpy="0 0 0" xyz="-0.12859312744504042 0.10167389824420814 0.028959375746381716"/>
+    <origin rpy="0 0 0" xyz="-0.12859312744504028 0.10517389824420881 0.02895937574638175"/>
     <mass value="0.21880690583277723"/>
     <inertia ixx="0.000235" ixy="1.1e-05" ixz="-7e-06" iyy="0.000273" iyz="0.0" izz="0.000371"/>
   </inertial>
   <visual>
-    <origin rpy="0 0 0" xyz="-0.333684 0.099028 -0.045405"/>
+    <origin rpy="0 0 0" xyz="-0.333684 0.102528 -0.048905"/>
     <geometry>
       <mesh filename="package://braco_description/meshes/punho_1.stl" scale="0.001 0.001 0.001"/>
@@ -238,5 +238,5 @@
   </visual>
   <collision>
-    <origin rpy="0 0 0" xyz="-0.333684 0.099028 -0.045405"/>
+    <origin rpy="0 0 0" xyz="-0.333684 0.102528 -0.048905"/>
     <geometry>
       <mesh filename="package://braco_description/meshes/punho_1.stl" scale="0.001 0.001 0.001"/>
@@ -246,10 +246,10 @@
 <link name="Center_arm_bearing_guide_clamp_v1_punho_1">
   <inertial>
-    <origin rpy="0 0 0" xyz="2.830437085266091e-07 0.0016578450305452658 2.542280482520365e-07"/>
+    <origin rpy="0 0 0" xyz="2.8304370869314255e-07 0.0016578450305454705 2.542280483353032e-07"/>
     <mass value="0.00026744770959091237"/>
     <inertia ixx="0.0" ixy="0.0" ixz="0.0" iyy="0.0" iyz="-0.0" izz="0.0"/>
   </inertial>
   <visual>
-    <origin rpy="0 0 0" xyz="-0.168543 -0.021709 -0.073405"/>
+    <origin rpy="0 0 0" xyz="-0.168543 -0.021709 -0.076905"/>
     <geometry>
       <mesh filename="package://braco_description/meshes/Center_arm_bearing_guide_clamp_v1_punho_1.stl" scale="0.001 0.001 0.001"/>
@@ -258,5 +258,5 @@
   </visual>
   <collision>
-    <origin rpy="0 0 0" xyz="-0.168543 -0.021709 -0.073405"/>
+    <origin rpy="0 0 0" xyz="-0.168543 -0.021709 -0.076905"/>
     <geometry>
       <mesh filename="package://braco_description/meshes/Center_arm_bearing_guide_clamp_v1_punho_1.stl" scale="0.001 0.001 0.001"/>
@@ -264,32 +264,12 @@
   </collision>
 </link>
-<link name="tampa_1">
-  <inertial>
-    <origin rpy="0 0 0" xyz="-6.348378147066116e-06 -1.751400612895522e-06 0.0014999999999999875"/>
-    <mass value="0.03288605303938267"/>
-    <inertia ixx="2.7e-05" ixy="0.0" ixz="-0.0" iyy="2.7e-05" iyz="0.0" izz="5.4e-05"/>
-  </inertial>
-  <visual>
-    <origin rpy="0 0 0" xyz="-0.0 0.0 -0.0655"/>
-    <geometry>
-      <mesh filename="package://braco_description/meshes/tampa_1.stl" scale="0.001 0.001 0.001"/>
-    </geometry>
-    <material name="silver"/>
-  </visual>
-  <collision>
-    <origin rpy="0 0 0" xyz="-0.0 0.0 -0.0655"/>
-    <geometry>
-      <mesh filename="package://braco_description/meshes/tampa_1.stl" scale="0.001 0.001 0.001"/>
-    </geometry>
-  </collision>
-</link>
 <link name="Base_servo_mount_left_1">
   <inertial>
-    <origin rpy="0 0 0" xyz="-0.015874540487837988 0.00020637077105250395 0.042452933406575036"/>
+    <origin rpy="0 0 0" xyz="-0.01587454048783796 0.00020637077105224721 0.042452933406575105"/>
     <mass value="0.04710420541299449"/>
     <inertia ixx="2.1e-05" ixy="0.0" ixz="0.0" iyy="3.9e-05" iyz="0.0" izz="2e-05"/>
   </inertial>
   <visual>
-    <origin rpy="0 0 0" xyz="-0.017324 -0.037609 -0.0685"/>
+    <origin rpy="0 0 0" xyz="-0.017324 -0.037609 -0.072"/>
     <geometry>
       <mesh filename="package://braco_description/meshes/Base_servo_mount_left_1.stl" scale="0.001 0.001 0.001"/>
@@ -298,5 +278,5 @@
   </visual>
   <collision>
-    <origin rpy="0 0 0" xyz="-0.017324 -0.037609 -0.0685"/>
+    <origin rpy="0 0 0" xyz="-0.017324 -0.037609 -0.072"/>
     <geometry>
       <mesh filename="package://braco_description/meshes/Base_servo_mount_left_1.stl" scale="0.001 0.001 0.001"/>
@@ -306,10 +286,10 @@
 <link name="Base_servo_mount_right_v1_1">
   <inertial>
-    <origin rpy="0 0 0" xyz="-0.015875047506617494 -0.00020585580724314517 0.04245293340657591"/>
+    <origin rpy="0 0 0" xyz="-0.015875047506617307 -0.00020585580724299946 0.042452933406575896"/>
     <mass value="0.04710420541299451"/>
     <inertia ixx="2.1e-05" ixy="-0.0" ixz="-0.0" iyy="3.9e-05" iyz="-0.0" izz="2e-05"/>
   </inertial>
   <visual>
-    <origin rpy="0 0 0" xyz="-0.01732 0.036811 -0.0685"/>
+    <origin rpy="0 0 0" xyz="-0.01732 0.036811 -0.072"/>
     <geometry>
       <mesh filename="package://braco_description/meshes/Base_servo_mount_right_v1_1.stl" scale="0.001 0.001 0.001"/>
@@ -318,5 +298,5 @@
   </visual>
   <collision>
-    <origin rpy="0 0 0" xyz="-0.01732 0.036811 -0.0685"/>
+    <origin rpy="0 0 0" xyz="-0.01732 0.036811 -0.072"/>
     <geometry>
       <mesh filename="package://braco_description/meshes/Base_servo_mount_right_v1_1.stl" scale="0.001 0.001 0.001"/>
@@ -324,32 +304,12 @@
   </collision>
 </link>
-<link name="NEMA17_-_Motor_de_passo_v1_1">
-  <inertial>
-    <origin rpy="0 0 0" xyz="-1.4033444489162447e-09 -6.644229439427179e-05 0.02054905046992122"/>
-    <mass value="0.06671740009958446"/>
-    <inertia ixx="1.9e-05" ixy="0.0" ixz="0.0" iyy="1.9e-05" iyz="-0.0" izz="1.9e-05"/>
-  </inertial>
-  <visual>
-    <origin rpy="0 0 0" xyz="-0.0 -0.0 -0.0"/>
-    <geometry>
-      <mesh filename="package://braco_description/meshes/NEMA17_-_Motor_de_passo_v1_1.stl" scale="0.001 0.001 0.001"/>
-    </geometry>
-    <material name="silver"/>
-  </visual>
-  <collision>
-    <origin rpy="0 0 0" xyz="-0.0 -0.0 -0.0"/>
-    <geometry>
-      <mesh filename="package://braco_description/meshes/NEMA17_-_Motor_de_passo_v1_1.stl" scale="0.001 0.001 0.001"/>
-    </geometry>
-  </collision>
-</link>
 <link name="corpo_garra_1">
   <inertial>
-    <origin rpy="0 0 0" xyz="0.036900222351620715 3.972525986601586e-09 -0.004369638500211437"/>
+    <origin rpy="0 0 0" xyz="0.03690022235162099 3.972526448471712e-09 -0.004369638500211395"/>
     <mass value="0.0475742677792808"/>
     <inertia ixx="2e-05" ixy="-0.0" ixz="2e-06" iyy="5.2e-05" iyz="0.0" izz="4.3e-05"/>
   </inertial>
   <visual>
-    <origin rpy="0 0 0" xyz="-0.255193 -0.000397 -0.073089"/>
+    <origin rpy="0 0 0" xyz="-0.255193 -0.000397 -0.076589"/>
     <geometry>
       <mesh filename="package://braco_description/meshes/corpo_garra_1.stl" scale="0.001 0.001 0.001"/>
@@ -358,5 +318,5 @@
   </visual>
   <collision>
-    <origin rpy="0 0 0" xyz="-0.255193 -0.000397 -0.073089"/>
+    <origin rpy="0 0 0" xyz="-0.255193 -0.000397 -0.076589"/>
     <geometry>
       <mesh filename="package://braco_description/meshes/corpo_garra_1.stl" scale="0.001 0.001 0.001"/>
@@ -366,10 +326,10 @@
 <link name="Bearing_guide_v1_1">
   <inertial>
-    <origin rpy="0 0 0" xyz="-3.61286664807281e-07 3.972064047520849e-09 0.017250496155362616"/>
+    <origin rpy="0 0 0" xyz="-3.612866644742141e-07 3.972064578563073e-09 0.0172504961553627"/>
     <mass value="0.0016815613439380714"/>
-    <inertia ixx="0.0" ixy="0.0" ixz="-0.0" iyy="0.0" iyz="-0.0" izz="0.0"/>
-  </inertial>
-  <visual>
-    <origin rpy="0 0 0" xyz="-0.329943 -0.000397 -0.055839"/>
+    <inertia ixx="0.0" ixy="0.0" ixz="0.0" iyy="0.0" iyz="-0.0" izz="0.0"/>
+  </inertial>
+  <visual>
+    <origin rpy="0 0 0" xyz="-0.329943 -0.000397 -0.059339"/>
     <geometry>
       <mesh filename="package://braco_description/meshes/Bearing_guide_v1_1.stl" scale="0.001 0.001 0.001"/>
@@ -378,5 +338,5 @@
   </visual>
   <collision>
-    <origin rpy="0 0 0" xyz="-0.329943 -0.000397 -0.055839"/>
+    <origin rpy="0 0 0" xyz="-0.329943 -0.000397 -0.059339"/>
     <geometry>
       <mesh filename="package://braco_description/meshes/Bearing_guide_v1_1.stl" scale="0.001 0.001 0.001"/>
@@ -386,10 +346,10 @@
 <link name="Bearing_top-bottom_bushing_v1_1">
   <inertial>
-    <origin rpy="0 0 0" xyz="-3.6128666519585906e-07 3.9724632054411076e-09 -0.0017495038446375955"/>
+    <origin rpy="0 0 0" xyz="-3.6128666475176985e-07 3.972463791398172e-09 -0.00174950384463754"/>
     <mass value="0.0016106179771745465"/>
     <inertia ixx="0.0" ixy="-0.0" ixz="0.0" iyy="0.0" iyz="0.0" izz="0.0"/>
   </inertial>
   <visual>
-    <origin rpy="0 0 0" xyz="-0.329943 -0.000397 -0.085339"/>
+    <origin rpy="0 0 0" xyz="-0.329943 -0.000397 -0.088839"/>
     <geometry>
       <mesh filename="package://braco_description/meshes/Bearing_top-bottom_bushing_v1_1.stl" scale="0.001 0.001 0.001"/>
@@ -398,5 +358,5 @@
   </visual>
   <collision>
-    <origin rpy="0 0 0" xyz="-0.329943 -0.000397 -0.085339"/>
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
Commit message: Manipulador sem o servo e o apoio esquerdo

File: braco_description/urdf/braco.xacro (robot description, xacro)
@@ -24,24 +24,4 @@
   </collision>
 </link>
-<link name="servo_left_1">
-  <inertial>
-    <origin rpy="0 0 0" xyz="-0.0014473150385015854 0.1421669334642504 -0.006915072172979028"/>
-    <mass value="0.25257832542625036"/>
-    <inertia ixx="6.8e-05" ixy="-0.0" ixz="0.0" iyy="4.4e-05" iyz="1e-06" izz="4.1e-05"/>
-  </inertial>
-  <visual>
-    <origin rpy="0 0 0" xyz="-0.002899 0.093141 -0.112109"/>
-    <geometry>
-      <mesh filename="package://braco_description/meshes/servo_left_1.stl" scale="0.001 0.001 0.001"/>
-    </geometry>
-    <material name="silver"/>
-  </visual>
-  <collision>
-    <origin rpy="0 0 0" xyz="-0.002899 0.093141 -0.112109"/>
-    <geometry>
-      <mesh filename="package://braco_description/meshes/servo_left_1.stl" scale="0.001 0.001 0.001"/>
-    </geometry>
-  </collision>
-</link>
 <link name="servo_right_1">
   <inertial>
@@ -264,24 +244,4 @@
   </collision>
 </link>
-<link name="Base_servo_mount_left_1">
-  <inertial>
-    <origin rpy="0 0 0" xyz="-0.01587454048783796 0.00020637077105224721 0.042452933406575105"/>
-    <mass value="0.04710420541299449"/>
-    <inertia ixx="2.1e-05" ixy="0.0" ixz="0.0" iyy="3.9e-05" iyz="0.0" izz="2e-05"/>
-  </inertial>
-  <visual>
-    <origin rpy="0 0 0" xyz="-0.017324 -0.037609 -0.072"/>
-    <geometry>
-      <mesh filename="package://braco_description/meshes/Base_servo_mount_left_1.stl" scale="0.001 0.001 0.001"/>
-    </geometry>
-    <material name="silver"/>
-  </visual>
-  <collision>
-    <origin rpy="0 0 0" xyz="-0.017324 -0.037609 -0.072"/>
-    <geometry>
-      <mesh filename="package://braco_description/meshes/Base_servo_mount_left_1.stl" scale="0.001 0.001 0.001"/>
-    </geometry>
-  </collision>
-</link>
 <link name="Base_servo_mount_right_v1_1">
   <inertial>
@@ -504,9 +464,4 @@
   </collision>
 </link>
-<joint name="Rigid28" type="fixed">
-  <origin rpy="0 0 0" xyz="-0.014425 -0.13075 0.040109"/>
-  <parent link="Base_servo_mount_left_1"/>
-  <child link="servo_left_1"/>
-</joint>
 <joint name="Rigid37" type="fixed">
   <origin rpy="0 0 0" xyz="-0.08132 0.13075 -0.039311"/>
@@ -566,9 +521,4 @@
   <parent link="Center_arm_bearing_guide_v1__1__1"/>
   <child link="Center_arm_bearing_guide_clamp_v1_punho_1"/>
-</joint>
-<joint name="Rigid77" type="fixed">
-  <origin rpy="0 0 0" xyz="0.017324 0.037609 0.069"/>
-  <parent link="tampa_1"/>
-  <child link="Base_servo_mount_left_1"/>
 </joint>
 <joint name="Rigid78" type="fixed">
