Commit message: Manipulador para teste de colisão com todas as partes

File: braco_v2_description/urdf/braco_v2.xacro (robot description, xacro)
@@ -6,5 +6,5 @@
 <link name="base_link">
   <inertial>
-    <origin rpy="0 0 0" xyz="0.0 4.884981308350689e-17 0.019999999999999983"/>
+    <origin rpy="0 0 0" xyz="0.0 4.4408920985006264e-17 0.019999999999999983"/>
     <mass value="0.4404041661434851"/>
     <inertia ixx="0.000423" ixy="0.0" ixz="-0.0" iyy="0.000423" iyz="0.0" izz="0.000728"/>
@@ -24,21 +24,361 @@
   </collision>
 </link>
-<link name="servo_left_1">
-  <inertial>
-    <origin rpy="0 0 0" xyz="-0.0014473150385015167 0.11316693346425025 -0.006915072172978931"/>
+<link name="Center_arm_v1_1">
+  <inertial>
+    <origin rpy="0 0 0" xyz="0.014277150157445656 0.009887184158138248 -0.05601557501701446"/>
+    <mass value="0.24743903954578314"/>
+    <inertia ixx="0.000535" ixy="0.0" ixz="0.000118" iyy="0.000605" iyz="-0.0" izz="0.000106"/>
+  </inertial>
+  <visual>
+    <origin rpy="0 0 0" xyz="-0.142342 0.011691 -0.205954"/>
+    <geometry>
+      <mesh filename="package://braco_v2_description/meshes/Center_arm_v1_1.stl" scale="0.001 0.001 0.001"/>
+    </geometry>
+    <material name="silver"/>
+  </visual>
+  <collision>
+    <origin rpy="0 0 0" xyz="-0.142342 0.011691 -0.205954"/>
+    <geometry>
+      <mesh filename="package://braco_v2_description/meshes/Center_arm_v1_1.stl" scale="0.001 0.001 0.001"/>
+    </geometry>
+  </collision>
+</link>
+<link name="Center_arm_bearing_guide_v1_1">
+  <inertial>
+    <origin rpy="0 0 0" xyz="-0.01039213224987559 0.003221962356880813 0.00600019094374038"/>
+    <mass value="0.0033035453927957375"/>
+    <inertia ixx="0.0" ixy="0.0" ixz="-0.0" iyy="0.0" iyz="-0.0" izz="0.0"/>
+  </inertial>
+  <visual>
+    <origin rpy="0 0 0" xyz="-0.152734 -0.008309 -0.199954"/>
+    <geometry>
+      <mesh filename="package://braco_v2_description/meshes/Center_arm_bearing_guide_v1_1.stl" scale="0.001 0.001 0.001"/>
+    </geometry>
+    <material name="silver"/>
+  </visual>
+  <collision>
+    <origin rpy="0 0 0" xyz="-0.152734 -0.008309 -0.199954"/>
+    <geometry>
+      <mesh filename="package://braco_v2_description/meshes/Center_arm_bearing_guide_v1_1.stl" scale="0.001 0.001 0.001"/>
+    </geometry>
+  </collision>
+</link>
+<link name="Center_arm_bearing_guide_v1__1__1">
+  <inertial>
+    <origin rpy="0 0 0" xyz="-0.0059998944503106 0.003221962356879297 -0.010392093645181094"/>
+    <mass value="0.0033035453927957375"/>
+    <inertia ixx="0.0" ixy="0.0" ixz="0.0" iyy="0.0" iyz="0.0" izz="0.0"/>
+  </inertial>
+  <visual>
+    <origin rpy="0 0 0" xyz="-0.178753 -0.008309 -0.10285"/>
+    <geometry>
+      <mesh filename="package://braco_v2_description/meshes/Center_arm_bearing_guide_v1__1__1.stl" scale="0.001 0.001 0.001"/>
+    </geometry>
+    <material name="silver"/>
+  </visual>
+  <collision>
+    <origin rpy="0 0 0" xyz="-0.178753 -0.008309 -0.10285"/>
+    <geometry>
+      <mesh filename="package://braco_v2_description/meshes/Center_arm_bearing_guide_v1__1__1.stl" scale="0.001 0.001 0.001"/>
+    </geometry>
+  </collision>
+</link>
+<link name="Center_arm_bearing_guide_clamp_v1_1">
+  <inertial>
+    <origin rpy="0 0 0" xyz="-1.322497980571491e-07 0.0016578450305448425 1.9094379913320303e-07"/>
+    <mass value="0.00026744770959091237"/>
+    <inertia ixx="0.0" ixy="-0.0" ixz="0.0" iyy="0.0" iyz="-0.0" izz="0.0"/>
+  </inertial>
+  <visual>
+    <origin rpy="0 0 0" xyz="-0.142342 -0.021709 -0.205954"/>
+    <geometry>
+      <mesh filename="package://braco_v2_description/meshes/Center_arm_bearing_guide_clamp_v1_1.stl" scale="0.001 0.001 0.001"/>
+    </geometry>
+    <material name="silver"/>
+  </visual>
+  <collision>
+    <origin rpy="0 0 0" xyz="-0.142342 -0.021709 -0.205954"/>
+    <geometry>
+      <mesh filename="package://braco_v2_description/meshes/Center_arm_bearing_guide_clamp_v1_1.stl" scale="0.001 0.001 0.001"/>
+    </geometry>
+  </collision>
+</link>
+<link name="servo_elbow_1">
+  <inertial>
+    <origin rpy="0 0 0" xyz="0.15754580602873644 0.20794860786324015 -0.030115300811952045"/>
+    <mass value="0.2525786066068201"/>
+    <inertia ixx="5.2e-05" ixy="-0.0" ixz="-1.4e-05" iyy="4.4e-05" iyz="-0.0" izz="5.7e-05"/>
+  </inertial>
+  <visual>
+    <origin rpy="0 0 0" xyz="0.022846 0.244866 -0.229657"/>
+    <geometry>
+      <mesh filename="package://braco_v2_description/meshes/servo_elbow_1.stl" scale="0.001 0.001 0.001"/>
+    </geometry>
+    <material name="silver"/>
+  </visual>
+  <collision>
+    <origin rpy="0 0 0" xyz="0.022846 0.244866 -0.229657"/>
+    <geometry>
+      <mesh filename="package://braco_v2_description/meshes/servo_elbow_1.stl" scale="0.001 0.001 0.001"/>
+    </geometry>
+  </collision>
+</link>
+<link name="servo_punho_rot_1">
+  <inertial>
+    <origin rpy="0 0 0" xyz="0.14034378523693494 -0.10986496796742812 -0.22086481094673482"/>
     <mass value="0.25257832542625036"/>
-    <inertia ixx="6.8e-05" ixy="-0.0" ixz="0.0" iyy="4.4e-05" iyz="1e-06" izz="4.1e-05"/>
-  </inertial>
-  <visual>
-    <origin rpy="0 0 0" xyz="-0.002899 0.064141 -0.083109"/>
-    <geometry>
-      <mesh filename="package://braco_v2_description/meshes/servo_left_1.stl" scale="0.001 0.001 0.001"/>
-    </geometry>
-    <material name="silver"/>
-  </visual>
-  <collision>
-    <origin rpy="0 0 0" xyz="-0.002899 0.064141 -0.083109"/>
-    <geometry>
-      <mesh filename="package://braco_v2_description/meshes/servo_left_1.stl" scale="0.001 0.001 0.001"/>
+    <inertia ixx="4.4e-05" ixy="-0.0" ixz="1e-06" iyy="6.8e-05" iyz="0.0" izz="4.1e-05"/>
+  </inertial>
+  <visual>
+    <origin rpy="0 0 0" xyz="-0.093832 -0.110262 -0.322983"/>
+    <geometry>
+      <mesh filename="package://braco_v2_description/meshes/servo_punho_rot_1.stl" scale="0.001 0.001 0.001"/>
+    </geometry>
+    <material name="silver"/>
+  </visual>
+  <collision>
+    <origin rpy="0 0 0" xyz="-0.093832 -0.110262 -0.322983"/>
+    <geometry>
+      <mesh filename="package://braco_v2_description/meshes/servo_punho_rot_1.stl" scale="0.001 0.001 0.001"/>
+    </geometry>
+  </collision>
+</link>
+<link name="servo_punho_xy_1">
+  <inertial>
+    <origin rpy="0 0 0" xyz="0.009976146320704926 -0.02522641850043935 -6.558513723775583e-08"/>
+    <mass value="0.25257832542625036"/>
+    <inertia ixx="4.1e-05" ixy="1e-06" ixz="0.0" iyy="4.4e-05" iyz="-0.0" izz="6.8e-05"/>
+  </inertial>
+  <visual>
+    <origin rpy="0 0 0" xyz="-0.172753 0.011691 -0.092458"/>
+    <geometry>
+      <mesh filename="package://braco_v2_description/meshes/servo_punho_xy_1.stl" scale="0.001 0.001 0.001"/>
+    </geometry>
+    <material name="silver"/>
+  </visual>
+  <collision>
+    <origin rpy="0 0 0" xyz="-0.172753 0.011691 -0.092458"/>
+    <geometry>
+      <mesh filename="package://braco_v2_description/meshes/servo_punho_xy_1.stl" scale="0.001 0.001 0.001"/>
+    </geometry>
+  </collision>
+</link>
+<link name="punho_1">
+  <inertial>
+    <origin rpy="0 0 0" xyz="-0.1328033049390942 0.12072689824420818 0.028960027873234748"/>
+    <mass value="0.21880690583277723"/>
+    <inertia ixx="0.000235" ixy="1.1e-05" ixz="-7e-06" iyy="0.000273" iyz="0.0" izz="0.000371"/>
+  </inertial>
+  <visual>
+    <origin rpy="0 0 0" xyz="-0.342104 0.118081 -0.064457"/>
+    <geometry>
+      <mesh filename="package://braco_v2_description/meshes/punho_1.stl" scale="0.001 0.001 0.001"/>
+    </geometry>
+    <material name="silver"/>
+  </visual>
+  <collision>
+    <origin rpy="0 0 0" xyz="-0.342104 0.118081 -0.064457"/>
+    <geometry>
+      <mesh filename="package://braco_v2_description/meshes/punho_1.stl" scale="0.001 0.001 0.001"/>
+    </geometry>
+  </collision>
+</link>
+<link name="Center_arm_bearing_guide_clamp_v1_punho_1">
+  <inertial>
+    <origin rpy="0 0 0" xyz="1.05549629869639e-07 0.0016578450305445892 -9.36450987448767e-08"/>
+    <mass value="0.00026744770959091237"/>
+    <inertia ixx="0.0" ixy="0.0" ixz="-0.0" iyy="0.0" iyz="-0.0" izz="0.0"/>
+  </inertial>
+  <visual>
+    <origin rpy="0 0 0" xyz="-0.172753 -0.021709 -0.092458"/>
+    <geometry>
+      <mesh filename="package://braco_v2_description/meshes/Center_arm_bearing_guide_clamp_v1_punho_1.stl" scale="0.001 0.001 0.001"/>
+    </geometry>
+    <material name="silver"/>
+  </visual>
+  <collision>
+    <origin rpy="0 0 0" xyz="-0.172753 -0.021709 -0.092458"/>
+    <geometry>
+      <mesh filename="package://braco_v2_description/meshes/Center_arm_bearing_guide_clamp_v1_punho_1.stl" scale="0.001 0.001 0.001"/>
+    </geometry>
+  </collision>
+</link>
+<link name="corpo_garra_1">
+  <inertial>
+    <origin rpy="0 0 0" xyz="0.03690104485756707 3.972525702432197e-09 -0.004369986373359419"/>
+    <mass value="0.0475742677792808"/>
+    <inertia ixx="2e-05" ixy="-0.0" ixz="2e-06" iyy="5.2e-05" iyz="0.0" izz="4.3e-05"/>
+  </inertial>
+  <visual>
+    <origin rpy="0 0 0" xyz="-0.259402 -0.000397 -0.092142"/>
+    <geometry>
+      <mesh filename="package://braco_v2_description/meshes/corpo_garra_1.stl" scale="0.001 0.001 0.001"/>
+    </geometry>
+    <material name="silver"/>
+  </visual>
+  <collision>
+    <origin rpy="0 0 0" xyz="-0.259402 -0.000397 -0.092142"/>
+    <geometry>
+      <mesh filename="package://braco_v2_description/meshes/corpo_garra_1.stl" scale="0.001 0.001 0.001"/>
+    </geometry>
+  </collision>
+</link>
+<link name="Bearing_guide_v1_1">
+  <inertial>
+    <origin rpy="0 0 0" xyz="4.6121928154452263e-07 3.97206351886387e-09 0.01725014828221419"/>
+    <mass value="0.0016815613439380714"/>
+    <inertia ixx="0.0" ixy="0.0" ixz="-0.0" iyy="0.0" iyz="-0.0" izz="0.0"/>
+  </inertial>
+  <visual>
+    <origin rpy="0 0 0" xyz="-0.334152 -0.000397 -0.074892"/>
+    <geometry>
+      <mesh filename="package://braco_v2_description/meshes/Bearing_guide_v1_1.stl" scale="0.001 0.001 0.001"/>
+    </geometry>
+    <material name="silver"/>
+  </visual>
+  <collision>
+    <origin rpy="0 0 0" xyz="-0.334152 -0.000397 -0.074892"/>
+    <geometry>
+      <mesh filename="package://braco_v2_description/meshes/Bearing_guide_v1_1.stl" scale="0.001 0.001 0.001"/>
+    </geometry>
+  </collision>
+</link>
+<link name="Bearing_top-bottom_bushing_v1_1">
+  <inertial>
+    <origin rpy="0 0 0" xyz="4.6121928093389997e-07 3.972462620622456e-09 -0.001749851717786216"/>
+    <mass value="0.0016106179771745465"/>
+    <inertia ixx="0.0" ixy="0.0" ixz="0.0" iyy="0.0" iyz="-0.0" izz="0.0"/>
+  </inertial>
+  <visual>
+    <origin rpy="0 0 0" xyz="-0.334152 -0.000397 -0.104392"/>
+    <geometry>
+      <mesh filename="package://braco_v2_description/meshes/Bearing_top-bottom_bushing_v1_1.stl" scale="0.001 0.001 0.001"/>
+    </geometry>
+    <material name="silver"/>
+  </visual>
+  <collision>
+    <origin rpy="0 0 0" xyz="-0.334152 -0.000397 -0.104392"/>
+    <geometry>
+      <mesh filename="package://braco_v2_description/meshes/Bearing_top-bottom_bushing_v1_1.stl" scale="0.001 0.001 0.001"/>
+    </geometry>
+  </collision>
+</link>
+<link name="Bearing_top-bottom_bushing_v1__1__1">
+  <inertial>
+    <origin rpy="0 0 0" xyz="4.612192812114557e-07 3.9724627058407465e-09 0.0017501482822140368"/>
+    <mass value="0.0016106179771745465"/>
+    <inertia ixx="0.0" ixy="0.0" ixz="0.0" iyy="0.0" iyz="-0.0" izz="0.0"/>
+  </inertial>
+  <visual>
+    <origin rpy="0 0 0" xyz="-0.334152 -0.000397 -0.079892"/>
+    <geometry>
+      <mesh filename="package://braco_v2_description/meshes/Bearing_top-bottom_bushing_v1__1__1.stl" scale="0.001 0.001 0.001"/>
+    </geometry>
+    <material name="silver"/>
+  </visual>
+  <collision>
+    <origin rpy="0 0 0" xyz="-0.334152 -0.000397 -0.079892"/>
+    <geometry>
+      <mesh filename="package://braco_v2_description/meshes/Bearing_top-bottom_bushing_v1__1__1.stl" scale="0.001 0.001 0.001"/>
+    </geometry>
+  </collision>
+</link>
+<link name="Bearing_center_bushing_v1_1">
+  <inertial>
+    <origin rpy="0 0 0" xyz="0.09827446121928143 0.04192300397246268 0.11753614828221406"/>
+    <mass value="0.0034513242368025996"/>
+    <inertia ixx="0.0" ixy="0.0" ixz="0.0" iyy="0.0" iyz="-0.0" izz="0.0"/>
+  </inertial>
+  <visual>
+    <origin rpy="0 0 0" xyz="-0.235878 0.041526 0.025394"/>
+    <geometry>
+      <mesh filename="package://braco_v2_description/meshes/Bearing_center_bushing_v1_1.stl" scale="0.001 0.001 0.001"/>
+    </geometry>
+    <material name="silver"/>
+  </visual>
+  <collision>
+    <origin rpy="0 0 0" xyz="-0.235878 0.041526 0.025394"/>
+    <geometry>
+      <mesh filename="package://braco_v2_description/meshes/Bearing_center_bushing_v1_1.stl" scale="0.001 0.001 0.001"/>
+    </geometry>
+  </collision>
+</link>
+<link name="servo_garra_1">
+  <inertial>
+    <origin rpy="0 0 0" xyz="0.053330533392260265 -0.018574770578143565 0.08636947229986802"/>
+    <mass value="0.25257832542625036"/>
+    <inertia ixx="4.1e-05" ixy="-0.0" ixz="1e-06" iyy="6.8e-05" iyz="0.0" izz="4.4e-05"/>
+  </inertial>
+  <visual>
+    <origin rpy="0 0 0" xyz="-0.245878 -0.018974 0.025394"/>
+    <geometry>
+      <mesh filename="package://braco_v2_description/meshes/servo_garra_1.stl" scale="0.001 0.001 0.001"/>
+    </geometry>
+    <material name="silver"/>
+  </visual>
+  <collision>
+    <origin rpy="0 0 0" xyz="-0.245878 -0.018974 0.025394"/>
+    <geometry>
+      <mesh filename="package://braco_v2_description/meshes/servo_garra_1.stl" scale="0.001 0.001 0.001"/>
+    </geometry>
+  </collision>
+</link>
+<link name="Gripper_120T_v1_1">
+  <inertial>
+    <origin rpy="0 0 0" xyz="0.010502843706276688 0.0181735244198357 0.006028625191617287"/>
+    <mass value="0.031315152970389164"/>
+    <inertia ixx="1e-05" ixy="-4e-06" ixz="-3e-06" iyy="4e-05" iyz="-0.0" izz="4.8e-05"/>
+  </inertial>
+  <visual>
+    <origin rpy="0 0 0" xyz="-0.334152 -0.000397 -0.083392"/>
+    <geometry>
+      <mesh filename="package://braco_v2_description/meshes/Gripper_120T_v1_1.stl" scale="0.001 0.001 0.001"/>
+    </geometry>
+    <material name="silver"/>
+  </visual>
+  <collision>
+    <origin rpy="0 0 0" xyz="-0.334152 -0.000397 -0.083392"/>
+    <geometry>
+      <mesh filename="package://braco_v2_description/meshes/Gripper_120T_v1_1.stl" scale="0.001 0.001 0.001"/>
+    </geometry>
+  </collision>
+</link>
+<link name="Gripper_72T_v1_1">
+  <inertial>
+    <origin rpy="0 0 0" xyz="0.020484421154321197 -0.01768686032720145 -0.0012214830647412217"/>
+    <mass value="0.0250024753894087"/>
+    <inertia ixx="4e-06" ixy="2e-06" ixz="2e-06" iyy="2e-05" iyz="-0.0" izz="2.2e-05"/>
+  </inertial>
+  <visual>
+    <origin rpy="0 0 0" xyz="-0.334152 -0.000397 -0.095892"/>
+    <geometry>
+      <mesh filename="package://braco_v2_description/meshes/Gripper_72T_v1_1.stl" scale="0.001 0.001 0.001"/>
+    </geometry>
+    <material name="silver"/>
+  </visual>
+  <collision>
+    <origin rpy="0 0 0" xyz="-0.334152 -0.000397 -0.095892"/>
+    <geometry>
+      <mesh filename="package://braco_v2_description/meshes/Gripper_72T_v1_1.stl" scale="0.001 0.001 0.001"/>
+    </geometry>
+  </collision>
+</link>
+<link name="Servo_gear_v1_1">
+  <inertial>
+    <origin rpy="0 0 0" xyz="4.926212099354288e-07 2.574818621269492e-07 0.0043180267545464834"/>
+    <mass value="0.010154744217590462"/>
+    <inertia ixx="1e-06" ixy="0.0" ixz="0.0" iyy="1e-06" iyz="0.0" izz="1e-06"/>
+  </inertial>
+  <visual>
+    <origin rpy="0 0 0" xyz="-0.289232 -0.000399 -0.086202"/>
+    <geometry>
+      <mesh filename="package://braco_v2_description/meshes/Servo_gear_v1_1.stl" scale="0.001 0.001 0.001"/>
+    </geometry>
+    <material name="silver"/>
+  </visual>
+  <collision>
+    <origin rpy="0 0 0" xyz="-0.289232 -0.000399 -0.086202"/>
+    <geometry>
+      <mesh filename="package://braco_v2_description/meshes/Servo_gear_v1_1.stl" scale="0.001 0.001 0.001"/>
     </geometry>
   </collision>
@@ -46,10 +386,10 @@
 <link name="servo_right_1">
   <inertial>
-    <origin rpy="0 0 0" xyz="0.06544272704404532 -0.11316641850044139 0.07250492782702289"/>
+    <origin rpy="0 0 0" xyz="0.045095727044045304 0.0126085814995585 0.08368692782702274"/>
     <mass value="0.25257832542625036"/>
     <inertia ixx="6.8e-05" ixy="-0.0" ixz="-0.0" iyy="4.4e-05" iyz="-1e-06" izz="4.1e-05"/>
   </inertial>
   <visual>
-    <origin rpy="0 0 0" xyz="0.064 -0.064939 -0.003689"/>
+    <origin rpy="0 0 0" xyz="0.043653 0.060836 0.007493"/>
     <geometry>
       <mesh filename="package://braco_v2_description/meshes/servo_right_1.stl" scale="0.001 0.001 0.001"/>
@@ -58,5 +398,5 @@
   </visual>
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